File: hardware/modules/CAN+Power/CAN+Power v0.1/CAN+Power v0.1.kicad_pcb (KiCad board)
At the start: 2 copper layers, 40 x 40 mm, 15 parts, among them J1 Conn_01x05_Male, J2 1, U1 SN65HVD230, U2 MC33063AD

Commit message: готова
Parts:
- removed Rterm1: 120 Ohm, Resistor_SMD:R_1206_3216Metric
- added REF**: , Resistor_SMD:R_1206_3216Metric, B.Cu at (148.7, 87.1)
- added REF**: , Resistor_SMD:R_1206_3216Metric, B.Cu at (148.7, 81.9)
- added REF**: SOT-23, Package_TO_SOT_SMD:SOT-23, B.Cu at (145.3, 84.5)
- added REF**: , Resistor_SMD:R_1206_3216Metric, B.Cu at (141.8, 86.8)
- added REF**: , Resistor_SMD:R_1206_3216Metric, B.Cu at (141.8, 82.2)
- moved U1 3.76 mm to (135.8, 84.5)
- moved Ct1 2.78 mm to (139.0, 107.8), turned to 270 degrees
- moved D1 2.51 mm to (141.4, 97.8), turned to 0 degrees
- moved J2 0.10 mm to (154.2, 93.1)
- turned L1 to 180 degrees
Connections:
- C1 pad 2: Net-(C1-Pad2) -> GND
- C2 pad 2: Net-(C1-Pad2) -> GND
- J2 pad 2: CANL -> CAN-
- J2 pad 3: CANH -> CAN+
- J2 pad 4: Net-(C1-Pad2) -> GND
- U1 pad 6: CANL -> (no net)
- U1 pad 7: CANH -> (no net)
Routing:
- net (no net): track 0.00 -> 24.6 mm, vias 0 -> 2
- net GND: track 7.40 -> 30.3 mm, vias 0 -> 6
- net CAN-: track 0.00 -> 10.3 mm
- net CAN+: track 0.00 -> 6.59 mm
- net CAN_TXD: track 14.7 -> 10.9 mm
- net CAN_RXD: track 14.4 -> 10.6 mm
- net MODE: track 20.6 -> 16.9 mm
- net Net-(D1-Pad1): track 17.9 -> 14.7 mm
- net 3.3+: track 65.7 -> 64.3 mm
- net Net-(Ct1-Pad1): track 5.17 -> 4.11 mm
- added copper zone on B.Cu, net GND

Commit message: плата готова и заказана
Parts:
- renumbered REF** to R3, REF** to R4, REF** to R5, REF** to R6, REF** to VD1
Routing:
- net CAN-: track 10.3 -> 5.65 mm
Other:
- board text added: "CAN+Power PCB v0.1"
- board text added: "spAm 2020"
Changed lines of the file:
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@@
   (general
     (thickness 1.6)
-    (drawings 6)
-    (tracks 111)
+    (drawings 8)
+    (tracks 103)
     (zones 0)
     (modules 19)
@@
       (outputformat 1)
       (mirror false)
-      (drillshape 1)
+      (drillshape 0)
       (scaleselection 1)
-      (outputdirectory ""))
+      (outputdirectory "fab/"))
   )
   (net 0 "")
@@
     (tags resistor)
     (attr smd)
-    (fp_text reference REF** (at 0 1.82 90) (layer B.SilkS)
+    (fp_text reference R5 (at 0 1.82 90) (layer B.SilkS)
       (effects (font (size 1 1) (thickness 0.15)) (justify mirror))
     )
@@
     (tags resistor)
     (attr smd)
-    (fp_text reference REF** (at 0 1.82 90) (layer B.SilkS)
+    (fp_text reference R6 (at 0 1.82 90) (layer B.SilkS)
       (effects (font (size 1 1) (thickness 0.15)) (justify mirror))
     )
@@
     (tags SOT-23)
     (attr smd)
-    (fp_text reference REF** (at 0 2.5) (layer B.SilkS)
+    (fp_text reference VD1 (at -0.5 2.45) (layer B.SilkS)
       (effects (font (size 1 1) (thickness 0.15)) (justify mirror))
     )
@@
     (tags resistor)
     (attr smd)
-    (fp_text reference REF** (at 0 1.82 90) (layer B.SilkS)
+    (fp_text reference R3 (at 0 1.82 90) (layer B.SilkS)
       (effects (font (size 1 1) (thickness 0.15)) (justify mirror))
     )
@@
     (tags resistor)
     (attr smd)
-    (fp_text reference REF** (at 0 1.82 90) (layer B.SilkS)
+    (fp_text reference R4 (at 0 1.82 90) (layer B.SilkS)
       (effects (font (size 1 1) (thickness 0.15)) (justify mirror))
     )
@@
     (descr "Through hole angled pin header, 1x05, 2.54mm pitch, 6mm pin length, single row")
     (tags "Through hole angled pin header THT 1x05 2.54mm single row")
-    (fp_text reference J1 (at 1.375 -1.5) (layer F.SilkS)
+    (fp_text reference J1 (at 1.45 -2.4) (layer F.SilkS)
       (effects (font (size 1 1) (thickness 0.15)))
     )
@@
     (tags "Diode SMA (DO-214AC)")
     (attr smd)
-    (fp_text reference D1 (at 5.08 -2.47) (layer F.SilkS)
+    (fp_text reference D1 (at -0.2 -2.5) (layer F.SilkS)
       (effects (font (size 1 1) (thickness 0.15)))
     )
@@
     (descr "Terminal Block Phoenix PT-1,5-4-5.0-H, 4 pins, pitch 5mm, size 20x9mm^2, drill diamater 1.3mm, pad diameter 2.6mm, see http://www.mouser.com/ds/2/324/ItemDetail_1935161-922578.pdf, script-generated using https://github.com/pointhi/kicad-footprint-generator/scripts/TerminalBlock_Phoenix")
     (tags "THT Terminal Block Phoenix PT-1,5-4-5.0-H pitch 5mm size 20x9mm^2 drill 1.3mm pad 2.6mm")
-    (fp_text reference J2 (at 10 -3.2 90) (layer F.SilkS)
+    (fp_text reference J2 (at -3.6 -4.15 180) (layer F.SilkS)
       (effects (font (size 1 1) (thickness 0.15)))
     )
@@
     (tags "capacitor electrolytic")
     (attr smd)
-    (fp_text reference С0 (at 0 -5.3) (layer F.SilkS)
+    (fp_text reference С0 (at 5.6 -2.65) (layer F.SilkS)
       (effects (font (size 1 1) (thickness 0.15)))
     )
@@
     (tags resistor)
     (attr smd)
-    (fp_text reference R2 (at 0 -1.82) (layer F.SilkS)
+    (fp_text reference R2 (at 0 1.65) (layer F.SilkS)
       (effects (font (size 1 1) (thickness 0.15)))
     )
@@
     (tags "Choke SMD")
     (attr smd)
-    (fp_text reference L1 (at 0 -6.35) (layer F.SilkS)
+    (fp_text reference L1 (at 0 6.65) (layer F.SilkS)
       (effects (font (size 1 1) (thickness 0.15)))
     )
@@
     (tags "capacitor electrolytic")
     (attr smd)
-    (fp_text reference C1 (at 0 -4.35) (layer F.SilkS)
+    (fp_text reference C1 (at 0.1 4.5) (layer F.SilkS)
       (effects (font (size 1 1) (thickness 0.15)))
     )
@@
       (rotate (xyz 0 0 0))
     )
+  )
+  (gr_text "spAm 2020" (at 138.85 78.25) (layer F.SilkS)
+    (effects (font (size 0.7 0.7) (thickness 0.1)))
+  )
+  (gr_text "CAN+Power PCB v0.1\n" (at 133.95 76.8) (layer F.SilkS)
+    (effects (font (size 1 1) (thickness 0.15)))
   )
   (dimension 40 (width 0.15) (layer Dwgs.User)
@@
   (segment (start 150.95 104.6) (end 147.86 104.6) (width 1) (layer F.Cu) (net 10))
   (segment (start 151.885 105.435) (end 151.05 104.6) (width 1) (layer F.Cu) (net 10))
-  (segment (start 148.7 87.95) (end 149.585 87.065) (width 0.7) (layer B.Cu) (net 12))
-  (segment (start 148.7 88.46) (end 148.7 87.835) (width 0.25) (layer B.Cu) (net 12))
-  (segment (start 149.585 87.1) (end 150.05 87.1) (width 0.7) (layer B.Cu) (net 12))
-  (segment (start 150.1 87.05) (end 150.65 86.5) (width 0.7) (layer B.Cu) (net 12))
-  (segment (start 150.7 86.4) (end 150.7 85.2) (width 0.7) (layer B.Cu) (net 12))
-  (segment (start 150.7 85.2) (end 151.2 84.7) (width 0.7) (layer B.Cu) (net 12))
-  (segment (start 151.2 84.7) (end 152.2 84.7) (width 0.7) (layer B.Cu) (net 12))
-  (segment (start 152.2 84.7) (end 152.8 85.3) (width 0.7) (layer B.Cu) (net 12))
-  (segment (start 152.8 86.65) (end 154.3 88.15) (width 0.7) (layer B.Cu) (net 12))
-  (segment (start 152.8 85.3) (end 152.8 86.6) (width 0.7) (layer B.Cu) (net 12))
+  (segment (start 153.84 88.46) (end 154.2 88.1) (width 0.25) (layer B.Cu) (net 12))
+  (segment (start 148.7 88.46) (end 153.84 88.46) (width 0.7) (layer B.Cu) (net 12))
   (segment (start 151.56 80.46) (end 148.7 80.46) (width 0.7) (layer B.Cu) (net 13))
   (segment (start 154.2 83.1) (end 151.56 80.46) (width 0.7) (layer B.Cu) (net 13))
@@
     (polygon
       (pts
-        (xy 160 115) (xy 120.05 115.05) (xy 119.95 75.1) (xy 119.95 75.05) (xy 160 75)
+        (xy 160 115) (xy 120.05 114.95) (xy 120 75.05) (xy 160 75.05)
       )
     )
